File: CC2500 Module.brd (EAGLE design)
At the start: 48.3 x 27.9 mm, 16 parts, among them IC1 CC2500

Commit message: Added Readme
Parts:
- IC1: device chipcon-ti:QLP-20 -> taylor:QLP-20
- R13: value 100R -> 330R
Changed lines of the file:
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@@
 <layer number="23" name="tOrigins" color="15" fill="1" visible="yes" active="yes"/>
 <layer number="24" name="bOrigins" color="15" fill="1" visible="yes" active="yes"/>
-<layer number="25" name="tNames" color="7" fill="1" visible="no" active="yes"/>
-<layer number="26" name="bNames" color="7" fill="1" visible="no" active="yes"/>
-<layer number="27" name="tValues" color="15" fill="1" visible="no" active="yes"/>
-<layer number="28" name="bValues" color="7" fill="1" visible="no" active="yes"/>
+<layer number="25" name="tNames" color="7" fill="1" visible="yes" active="yes"/>
+<layer number="26" name="bNames" color="7" fill="1" visible="yes" active="yes"/>
+<layer number="27" name="tValues" color="15" fill="1" visible="yes" active="yes"/>
+<layer number="28" name="bValues" color="7" fill="1" visible="yes" active="yes"/>
 <layer number="29" name="tStop" color="15" fill="5" visible="no" active="yes"/>
 <layer number="30" name="bStop" color="7" fill="6" visible="no" active="yes"/>
@@
 </autorouter>
 <elements>
-<element name="R13" library="SparkFun" package="0402-RES" value="100R" x="39.116" y="11.3665" rot="R270"/>
-<element name="IC1" library="chipcon-ti" package="QLP-20" value="CC2500" x="23.876" y="9.144" rot="R90"/>
+<element name="R13" library="SparkFun" package="0402-RES" value="330R" x="39.116" y="11.3665" rot="R270"/>
+<element name="IC1" library="taylor" package="QLP-20" value="CC2500" x="23.876" y="9.144" rot="R90"/>
 <element name="U$22" library="taylor" package="CC2500_FOLDED_DIPOLE_ANTENNA" value="ANTENNA_DIPOLE" x="24.13" y="27.94"/>
 <element name="U$23" library="taylor" package="5X3.2MM_SMD_XTAL" value="7A-26.000MAAJ-T" x="29.972" y="9.779" rot="R270"/>
