File: CC2500 Module.sch (EAGLE design)
At the start: 16 parts, among them IC1 CC2500

Commit message: Added Readme
Parts:
- IC1: device chipcon-ti:CC2500 -> Taylor:CC2500
- R13: value 100R -> 330R
Connections:
- net +3V3: now also IC1.AVDD@1, IC1.AVDD@2, IC1.AVDD@3, IC1.AVDD@4, IC1.DGUARD, IC1.DVDD; no longer IC1G$1.DGUARD, IC1P.AVDD@1, IC1P.AVDD@2, IC1P.AVDD@3, IC1P.AVDD@4, IC1P.DVDD
- net DCOUPL: now also IC1.DCOUPL; no longer IC1G$1.DCOUPL
- net GND: now also IC1.AGND, IC1.GND@1, IC1.GND@2; no longer IC1P.AGND, IC1P.GND@1, IC1P.GND@2
- net MISO: now also IC1.SO/GDO1; no longer IC1G$1.SO/GDO1
- net MOSI: now also IC1.SI; no longer IC1G$1.SI
- net N$13: now also IC1.RF-N; no longer IC1G$1.RF-N
- net N$15: now also IC1.XOSC-1; no longer IC1G$1.XOSC-1
- net N$20: now also IC1.XOSC-2; no longer IC1G$1.XOSC-2
- net N$23: now also IC1.RBIAS; no longer IC1G$1.RBIAS
- net N$8: now also IC1.RF-P; no longer IC1G$1.RF-P
- net RF_CS: now also IC1.CS; no longer IC1G$1.CS
- net RF_GDO0: now also IC1.GDO0; no longer IC1G$1.GDO0
- net RF_GDO2: now also IC1.GDO2; no longer IC1G$1.GDO2
- net SPCK: now also IC1.SCLK; no longer IC1G$1.SCLK
Changed lines of the file:
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@@
 </classes>
 <parts>
-<part name="R13" library="SparkFun" deviceset="RESISTOR" device="0402-RES" value="100R"/>
+<part name="R13" library="SparkFun" deviceset="RESISTOR" device="0402-RES" value="330R"/>
 <part name="+3V21" library="supply1" deviceset="+3V3" device=""/>
-<part name="IC1" library="chipcon-ti" deviceset="CC2500" device=""/>
+<part name="IC1" library="Taylor" deviceset="CC2500" device=""/>
 <part name="U$22" library="taylor" deviceset="ANTENNA_DIPOLE" device=""/>
 <part name="GND30" library="SparkFun" deviceset="GND" device=""/>
